Commit message: Add options to not use a gripper
Problem:
* The interfaces assume a gripper is available, and throw errors when
  the hardware does not have the gripper motor

Solution:
* Added a flag to indicate whether the gripper is available. Gripper IO
  is optional based on this flag

Test: Tested on r5 without gripper

File: models/arx5_no_gripper.urdf (robot description, URDF)
Before this commit: robot arx5_gopro, 8 links, 7 joints
Links:
- link link6: mass 0.030 -> 0.14
Joints:
- joint gripper_fixed_joint: origin xyz=0.225 0.0 0.0 rpy=0 0 0 -> xyz=0.185 0.0 0.0 rpy=0 0 0
