Commit message: Update urdf file (without gopro)

File: models/arx5.urdf (robot description, URDF)
Before this commit: robot ultron_v1.1_aa, 7 links, 6 joints
Links:
- added link gripper_dummy_link, mass 0.0
- link link6: mass 1.010000 -> 0.581000
Joints:
- added joint gripper_fixed_joint: type fixed, parent link6, child gripper_dummy_link, origin xyz=0.145 0.0 0.0 rpy=0 0 0
- joint joint2: limit (none) -> lower=0 upper=3.14 effort=100 velocity=1000; type fixed -> revolute
- joint joint3: limit lower=-10 upper=10 effort=100 velocity=1000 -> lower=-0 upper=3.14 effort=100 velocity=1000
- joint joint4: limit lower=-10 upper=10 effort=100 velocity=1000 -> lower=-1.67 upper=1.67 effort=100 velocity=1000
- joint joint5: limit lower=-10 upper=10 effort=100 velocity=1000 -> lower=-1.67 upper=1.67 effort=100 velocity=1000
- joint joint6: limit lower=-10 upper=10 effort=100 velocity=1000 -> lower=-1.57 upper=1.57 effort=100 velocity=1000

Commit message: Fix urdf and update README

File: models/arx5.urdf (robot description, URDF)
Before this commit: robot ultron_v1.1_aa, 8 links, 7 joints
Links:
- link base_link: mass 0.44038 -> 0.428
- link link1: mass 0.060835 -> 0.064
- link link2: mass 1.0733 -> 1.165
- link link3: mass 0.4994 -> 0.546; geometry collision cylinder length=0.15 radius=0.02; visual mesh filename=./meshes/link3.STL
- link link4: geometry collision cylinder length=0.05 radius=0.025; visual mesh filename=./meshes/link4.STL
- link link5: mass 0.60236 -> 0.655; geometry collision cylinder length=0.025 radius=0.02; visual mesh filename=./meshes/link5.STL
Joints:
- joint joint3: limit lower=-0 upper=3.14 effort=100 velocity=1000 -> lower=0 upper=3.14 effort=30 velocity=10
- joint joint4: limit lower=-1.67 upper=1.67 effort=100 velocity=1000 -> lower=-1.57079632679 upper=1.57079632679 effort=30 velocity=10

File: models/arx5_gopro.urdf (robot description, URDF)
Before this commit: robot arx5_gopro, 8 links, 7 joints
Joints:
- joint joint4: limit lower=-1.57079632679  upper=1.57079632679  effort=30 velocity=10 -> lower=-1.57079632679 upper=1.57079632679 effort=30 velocity=10

Commit message: Update solver with multiple DoF

File: models/arx5.urdf (robot description, URDF)
Before this commit: robot ultron_v1.1_aa, 8 links, 7 joints
Links:
- removed link gripper_dummy_link
- added link eef_link, mass 0.0
Joints:
- joint gripper_fixed_joint: child gripper_dummy_link -> eef_link

File: models/arx5_gopro.urdf (robot description, URDF)
Before this commit: robot arx5_gopro, 8 links, 7 joints
Links:
- removed link gripper_dummy_link
- added link eef_link, mass 0.0001
Joints:
- joint gripper_fixed_joint: child gripper_dummy_link -> eef_link

File: models/arx5_no_gripper.urdf (robot description, URDF)
Before this commit: robot arx5_gopro, 8 links, 7 joints
Links:
- removed link gripper_dummy_link
- added link eef_link, mass 0.0
Joints:
- joint gripper_fixed_joint: child gripper_dummy_link -> eef_link
